File: differentiator_trimable.kicad_sch (KiCad schematic)
At the start: 0 parts

Commit message: Added spice/ submodule and high level schematic
Parts:
- added C1: 100p, symbol Device:C
- added R1: 150 R to 1K, symbol Device:R_Variable_US
- added R2: 50, symbol Device:R_US
Connections:
- new net GND: R2.2
- new net differ_in: C1.1, R1.1
- new net differ_out: C1.2, R1.2, R2.1
Other:
- note added: "An upstream pole with time constant τ_{u} gets cancelled if τ_{u} = τ_{pz} = R_{1}C_{1}"
- note added: "Make τ_{pz} adjustable from 15 ns to 100 ns and τ_{o} nominally 5 ns, but would be as low as 3.75 ns for τ_{pz} = 15 ns."
- note added: "The remaining output pole is at τ_{o} = R_{1}C_{1} || R_{2}C_{2} If R_{1}C_{1} >> R_{2}C_{1}, then τ_{o} ≅ R_{2}C_{1}"
Changed lines of the file:
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@@
     (company "HugonLabs")
+  )
+  (junction (at 34.29 55.88) (diameter 0) (color 0 0 0 0)
+  )
+  (junction (at 55.88 68.58) (diameter 0) (color 0 0 0 0)
+  )
+  (junction (at 55.88 55.88) (diameter 0) (color 0 0 0 0)
+  )
+  (wire (pts (xy 20.32 55.88) (xy 34.29 55.88))
+    (stroke (width 0) (type default) (color 0 0 0 0))
+  )
+  (wire (pts (xy 55.88 55.88) (xy 55.88 68.58))
+    (stroke (width 0) (type default) (color 0 0 0 0))
+  )
+  (wire (pts (xy 34.29 55.88) (xy 34.29 68.58))
+    (stroke (width 0) (type default) (color 0 0 0 0))
+  )
+  (wire (pts (xy 55.88 55.88) (xy 73.66 55.88))
+    (stroke (width 0) (type default) (color 0 0 0 0))
+  )
+  (wire (pts (xy 46.99 55.88) (xy 55.88 55.88))
+    (stroke (width 0) (type default) (color 0 0 0 0))
+  )
+  (wire (pts (xy 34.29 68.58) (xy 39.37 68.58))
+    (stroke (width 0) (type default) (color 0 0 0 0))
+  )
+  (wire (pts (xy 34.29 55.88) (xy 39.37 55.88))
+    (stroke (width 0) (type default) (color 0 0 0 0))
+  )
+  (wire (pts (xy 46.99 68.58) (xy 55.88 68.58))
+    (stroke (width 0) (type default) (color 0 0 0 0))
+  )
+  (text "Make τ_{pz} adjustable from 15 ns to 100 ns\nand τ_{o} nominally 5 ns, \nbut would be as low as 3.75 ns for τ_{pz} = 15 ns."
+    (at 17.78 38.1 0)
+    (effects (font (size 1.27 1.27)) (justify left bottom))
+  )
+  (text "An upstream pole with time constant τ_{u}\ngets cancelled if τ_{u} = τ_{pz} = R_{1}C_{1}"
+    (at 17.78 21.59 0)
+    (effects (font (size 1.27 1.27)) (justify left bottom))
+  )
+  (text "The remaining output pole is at τ_{o} = R_{1}C_{1} || R_{2}C_{2}\nIf R_{1}C_{1} >> R_{2}C_{1}, then τ_{o} ≅ R_{2}C_{1}"
+    (at 17.78 29.21 0)
+    (effects (font (size 1.27 1.27)) (justify left bottom))
+  )
+  (label "differ_in" (at 20.32 55.88 0)
+    (effects (font (size 1.27 1.27)) (justify left bottom))
+  )
+  (label "differ_out" (at 73.66 55.88 180)
+    (effects (font (size 1.27 1.27)) (justify right bottom))
+  )
+  (symbol (lib_id "Device:C") (at 43.18 55.88 90) (unit 1)
+    (in_bom yes) (on_board yes) (fields_autoplaced)
+    (property "Reference" "C1" (id 0) (at 43.18 48.26 90))
+    (property "Value" "100p" (id 1) (at 43.18 50.8 90))
+    (property "Footprint" "" (id 2) (at 46.99 54.9148 0)
+      (effects (font (size 1.27 1.27)) hide)
+    )
+    (property "Datasheet" "~" (id 3) (at 43.18 55.88 0)
+      (effects (font (size 1.27 1.27)) hide)
+    )
+    (pin "1")
+    (pin "2")
+  )
+  (symbol (lib_id "Device:R_Variable_US") (at 43.18 68.58 90) (unit 1)
+    (in_bom yes) (on_board yes) (fields_autoplaced)
+    (property "Reference" "R1" (id 0) (at 43.1419 60.96 90))
+    (property "Value" "150 R to 1K" (id 1) (at 43.1419 63.5 90))
+    (property "Footprint" "" (id 2) (at 43.18 70.358 90)
+      (effects (font (size 1.27 1.27)) hide)
+    )
+    (property "Datasheet" "~" (id 3) (at 43.18 68.58 0)
+      (effects (font (size 1.27 1.27)) hide)
+    )
+    (pin "1")
+    (pin "2")
+  )
+  (symbol (lib_id "power:GND") (at 55.88 76.2 0) (unit 1)
+    (in_bom yes) (on_board yes) (fields_autoplaced)
+    (property "Reference" "#PWR01" (id 0) (at 55.88 82.55 0)
+      (effects (font (size 1.27 1.27)) hide)
+    )
+    (property "Value" "GND" (id 1) (at 55.88 81.28 0))
+    (property "Footprint" "" (id 2) (at 55.88 76.2 0)
+      (effects (font (size 1.27 1.27)) hide)
+    )
+    (property "Datasheet" "" (id 3) (at 55.88 76.2 0)
+      (effects (font (size 1.27 1.27)) hide)
+    )
+    (pin "1")
+  )
+  (symbol (lib_id "Device:R_US") (at 55.88 72.39 0) (unit 1)
+    (in_bom yes) (on_board yes) (fields_autoplaced)
+    (property "Reference" "R2" (id 0) (at 58.42 71.1199 0)
+      (effects (font (size 1.27 1.27)) (justify left))
+    )
+    (property "Value" "50" (id 1) (at 58.42 73.6599 0)
+      (effects (font (size 1.27 1.27)) (justify left))
+    )
+    (property "Footprint" "" (id 2) (at 56.896 72.644 90)
+      (effects (font (size 1.27 1.27)) hide)
+    )
+    (property "Datasheet" "~" (id 3) (at 55.88 72.39 0)
+      (effects (font (size 1.27 1.27)) hide)
+    )
+    (pin "1")
+    (pin "2")
   )
   (sheet_instances
     (path "/" (page "1"))
   )
+  (symbol_instances
+    (path "/ed7f23d8-d2f8-4b40-8e90-ab4c922c2923"
+      (reference "#PWR01") (unit 1) (value "GND") (footprint "")
+    )
+    (path "/04d63568-b245-4606-a828-e095e69c6f98"
+      (reference "C1") (unit 1) (value "100p") (footprint "")
+    )
+    (path "/391d54e9-04b9-4851-9853-e5856b65c845"
+      (reference "R1") (unit 1) (value "150 R to 1K") (footprint "")
+    )
+    (path "/f7560940-4a3c-481c-9570-70324617c5fa"
+      (reference "R2") (unit 1) (value "50") (footprint "")
+    )
+  )
 )
